File: BMS.sch (KiCad schematic (older format))
At the start: 122 parts, among them J1 Conn_01x10_Male, J2 Conn_01x10_Male, J3 Conn_01x01_Male, J4 Conn_01x03_Male, J5 Conn_01x05_Male, J6 Conn_01x01_Male, J7 Conn_01x03_Male, J8 Conn_01x01_Male, J9 Conn_01x01_Male, Q1 BSS308PE, Q10 BSS308PE, Q11 BSS308PE, Q12 BSS308PE, Q13 BSS308PE, Q14 BSS308PE, Q15 BSS308PE, Q16 BSS308PE, Q17 BSS308PE, Q18 BSS308PE, Q19 BCP56, Q2 BSS308PE, Q20 IPT012N08N5, Q21 IPT012N08N5, Q3 BSS308PE, Q4 BSS308PE, Q5 BSS308PE, Q6 BSS308PE, Q7 BSS308PE, Q8 BSS308PE, Q9 BSS308PE, U1 LTC6813-1, U2 ACS758xCB-150B-PSS, U3 ACS758xCB-150B-PSS

Commit message: Remove diode on charge input
Parts:
- removed D1: C5D50065D, Package_TO_SOT_THT:TO-247-3_Vertical, symbol Diode:C5D50065D
- C23: value 100nF -> 100n
- R57, R59: value R -> 1k
Connections:
- wire segments 506 -> 501
Other:
- moved on the sheet: J8
Changed lines of the file:
@@
 P 12150 3900
 F 0 "C23" H 12265 3946 50  0000 L CNN
-F 1 "100nF" H 12265 3855 50  0000 L CNN
+F 1 "100n" H 12265 3855 50  0000 L CNN
 F 2 "Capacitor_SMD:C_0805_2012Metric_Pad1.15x1.40mm_HandSolder" H 12188 3750 50  0001 C CNN
 F 3 "~" H 12150 3900 50  0001 C CNN
@@
 	11300 5300 11300 5550
 $Comp
-L Device:R R63
-U 1 1 5E45713F
-P 12400 5350
-F 0 "R63" V 12193 5350 50  0000 C CNN
-F 1 "R" V 12284 5350 50  0000 C CNN
-F 2 "Resistor_SMD:R_0805_2012Metric_Pad1.15x1.40mm_HandSolder" V 12330 5350 50  0001 C CNN
-F 3 "~" H 12400 5350 50  0001 C CNN
-	1    12400 5350
-	0    1    1    0
-$EndComp
-$Comp
 L power:VCC #PWR021
 U 1 1 5E4581B1
@@
 P 11000 5400
 F 0 "R57" V 10793 5400 50  0000 C CNN
-F 1 "R" V 10884 5400 50  0000 C CNN
+F 1 "1k" V 10884 5400 50  0000 C CNN
 F 2 "Resistor_SMD:R_0805_2012Metric_Pad1.15x1.40mm_HandSolder" V 10930 5400 50  0001 C CNN
 F 3 "~" H 11000 5400 50  0001 C CNN
@@
 P 11350 5700
 F 0 "R59" V 11557 5700 50  0000 C CNN
-F 1 "R" V 11466 5700 50  0000 C CNN
+F 1 "1k" V 11466 5700 50  0000 C CNN
 F 2 "Resistor_SMD:R_0805_2012Metric_Pad1.15x1.40mm_HandSolder" V 11280 5700 50  0001 C CNN
 F 3 "~" H 11350 5700 50  0001 C CNN
@@
 Wire Wire Line
 	11100 2800 11100 2400
-$Comp
-L Diode:C5D50065D D1
-U 1 1 5E712BA5
-P 13400 1450
-F 0 "D1" H 13400 1134 50  0000 C CNN
-F 1 "C5D50065D" H 13400 1225 50  0000 C CNN
-F 2 "Package_TO_SOT_THT:TO-247-3_Vertical" H 13400 1275 50  0001 C CNN
-F 3 "https://www.wolfspeed.com/media/downloads/111/C5D50065D.pdf" H 13400 1450 50  0001 C CNN
-	1    13400 1450
-	-1   0    0    1
-$EndComp
-Wire Wire Line
-	13600 1350 13750 1350
-Wire Wire Line
-	13750 1350 13750 1450
-Wire Wire Line
-	13750 1550 13600 1550
-Connection ~ 13750 1450
-Wire Wire Line
-	13750 1450 13750 1550
 Wire Wire Line
 	11850 1450 11200 1450
@@
 	12400 1450 12550 1450
 Connection ~ 12400 1450
-Wire Wire Line
-	12950 1450 13200 1450
 $Comp
 L Sensor_Current:ACS758xCB-150B-PSS U3
@@
 L Connector:Conn_01x01_Male J8
 U 1 1 5E67882E
-P 14050 1450
-F 0 "J8" H 14022 1382 50  0000 R CNN
-F 1 "Conn_01x01_Male" H 14022 1473 50  0000 R CNN
-F 2 "TestPoint:TestPoint_Pad_4.0x4.0mm" H 14050 1450 50  0001 C CNN
-F 3 "~" H 14050 1450 50  0001 C CNN
-	1    14050 1450
+P 13700 1450
+F 0 "J8" H 13672 1382 50  0000 R CNN
+F 1 "Conn_01x01_Male" H 13672 1473 50  0000 R CNN
+F 2 "TestPoint:TestPoint_Pad_4.0x4.0mm" H 13700 1450 50  0001 C CNN
+F 3 "~" H 13700 1450 50  0001 C CNN
+	1    13700 1450
 	-1   0    0    1
 $EndComp
@@
 $EndComp
 Wire Wire Line
-	13750 1450 13850 1450
-Wire Wire Line
 	10850 1450 11000 1450
 Wire Wire Line
@@
 Wire Wire Line
 	8650 4550 8700 4550
+$Comp
+L Device:R R63
+U 1 1 5E45713F
+P 12400 5350
+F 0 "R63" V 12193 5350 50  0000 C CNN
+F 1 "R" V 12284 5350 50  0000 C CNN
+F 2 "Resistor_SMD:R_0805_2012Metric_Pad1.15x1.40mm_HandSolder" V 12330 5350 50  0001 C CNN
+F 3 "~" H 12400 5350 50  0001 C CNN
+	1    12400 5350
+	0    1    1    0
+$EndComp
+Wire Wire Line
+	12950 1450 13500 1450
 $EndSCHEMATC

Commit message: backup
Parts:
- R63: footprint Resistor_SMD:R_0805_2012Metric_Pad1.15x1.40mm_HandSolder -> Resistor_SMD:R_1206_3216Metric_Pad1.42x1.75mm_HandSolder
Connections:
- net GND: now also J3.1 (Pin_1), U2.5 (IP-)
- net VPP: now also J1.2 (Pin_2), Q1.2 (S), R19.2, R20.2; no longer C1.2, R19.1, U1.1 (V+)
- net at U1.39 (GPIO1): now also U3.3 (VIOUT); no longer U2.3 (VIOUT)
- net at U1.40 (GPIO2): now also U2.3 (VIOUT); no longer U3.3 (VIOUT)
- new net: C1.2, R19.1, U1.1 (V+)
Other:
- moved on the sheet: J3
Changed lines of the file:
@@
 L power:VPP #PWR03
 U 1 1 5E42E243
-P 8550 4400
-F 0 "#PWR03" H 8550 4250 50  0001 C CNN
-F 1 "VPP" H 8565 4573 50  0000 C CNN
-F 2 "" H 8550 4400 50  0001 C CNN
-F 3 "" H 8550 4400 50  0001 C CNN
-	1    8550 4400
+P 3700 1200
+F 0 "#PWR03" H 3700 1050 50  0001 C CNN
+F 1 "VPP" H 3715 1373 50  0000 C CNN
+F 2 "" H 3700 1200 50  0001 C CNN
+F 3 "" H 3700 1200 50  0001 C CNN
+	1    3700 1200
 	1    0    0    -1
 $EndComp
@@
 Connection ~ 4300 1350
 Wire Wire Line
-	4300 1350 3500 1350
+	4300 1350 4000 1350
 Wire Wire Line
 	5150 900  5150 700
@@
 $EndComp
 Wire Wire Line
-	10800 7200 13950 7200
-Wire Wire Line
-	13950 7200 13950 2800
-Wire Wire Line
 	13950 2800 11100 2800
 Wire Wire Line
@@
 	6900 6050 8700 6050
 Wire Wire Line
-	15000 1650 15000 7300
-Wire Wire Line
-	15000 7300 10800 7300
+	15000 1650 15000 7200
 Wire Wire Line
 	11700 3650 11700 3800
@@
 L Connector:Conn_01x01_Male J3
 U 1 1 5E67770D
-P 10650 1450
-F 0 "J3" H 10758 1631 50  0000 C CNN
-F 1 "Conn_01x01_Male" H 10758 1540 50  0000 C CNN
-F 2 "TestPoint:TestPoint_Pad_4.0x4.0mm" H 10650 1450 50  0001 C CNN
-F 3 "~" H 10650 1450 50  0001 C CNN
-	1    10650 1450
+P 10450 1450
+F 0 "J3" H 10558 1631 50  0000 C CNN
+F 1 "Conn_01x01_Male" H 10558 1540 50  0000 C CNN
+F 2 "TestPoint:TestPoint_Pad_4.0x4.0mm" H 10450 1450 50  0001 C CNN
+F 3 "~" H 10450 1450 50  0001 C CNN
+	1    10450 1450
 	1    0    0    -1
 $EndComp
@@
 $EndComp
 Wire Wire Line
-	10850 1450 11000 1450
-Wire Wire Line
 	11000 1450 11000 1600
 $Comp
@@
 	1    0    0    -1
 $EndComp
-Wire Wire Line
-	8400 4550 8550 4550
 $Comp
 L power:PWR_FLAG #FLG01
 U 1 1 5EEBA562
-P 8650 4050
-F 0 "#FLG01" H 8650 4125 50  0001 C CNN
-F 1 "PWR_FLAG" H 8650 4223 50  0000 C CNN
-F 2 "" H 8650 4050 50  0001 C CNN
-F 3 "~" H 8650 4050 50  0001 C CNN
-	1    8650 4050
+P 4000 1200
+F 0 "#FLG01" H 4000 1275 50  0001 C CNN
+F 1 "PWR_FLAG" H 4000 1373 50  0000 C CNN
+F 2 "" H 4000 1200 50  0001 C CNN
+F 3 "~" H 4000 1200 50  0001 C CNN
+	1    4000 1200
 	1    0    0    -1
 $EndComp
 Wire Wire Line
 	4300 900  4800 900
-Wire Wire Line
-	8550 4400 8550 4550
-Connection ~ 8550 4550
-Wire Wire Line
-	8550 4550 8650 4550
-Wire Wire Line
-	8650 4050 8650 4550
-Connection ~ 8650 4550
-Wire Wire Line
-	8650 4550 8700 4550
 $Comp
 L Device:R R63
@@
 F 0 "R63" V 12193 5350 50  0000 C CNN
 F 1 "R" V 12284 5350 50  0000 C CNN
-F 2 "Resistor_SMD:R_0805_2012Metric_Pad1.15x1.40mm_HandSolder" V 12330 5350 50  0001 C CNN
+F 2 "Resistor_SMD:R_1206_3216Metric_Pad1.42x1.75mm_HandSolder" V 12330 5350 50  0001 C CNN
 F 3 "~" H 12400 5350 50  0001 C CNN
 	1    12400 5350
@@
 Wire Wire Line
 	12950 1450 13500 1450
+Wire Wire Line
+	13950 7300 10800 7300
+Wire Wire Line
+	13950 2800 13950 7300
+Wire Wire Line
+	10800 7200 15000 7200
+Wire Wire Line
+	10650 1450 10750 1450
+Wire Wire Line
+	10750 1450 10750 2000
+Connection ~ 10750 1450
+Wire Wire Line
+	10750 1450 11000 1450
+Connection ~ 10750 2000
+Wire Wire Line
+	8400 4550 8700 4550
+Wire Wire Line
+	4000 1200 4000 1350
+Connection ~ 4000 1350
+Wire Wire Line
+	4000 1350 3700 1350
+Wire Wire Line
+	3700 1200 3700 1350
+Connection ~ 3700 1350
+Wire Wire Line
+	3700 1350 3500 1350
 $EndSCHEMATC

Commit message: First routing
Parts:
- added J4: Conn_01x08_Male, Connector_PinHeader_2.54mm:PinHeader_1x08_P2.54mm_Vertical, symbol Connector:Conn_01x08_Male
- renumbered J9 to J10, J4 to J5, J5 to J6, J6 to J7, J7 to J9
Connections:
- net GND: now also J4.1 (Pin_1)
- net at U1.41 (GPIO3): now also J4.8 (Pin_8)
- net at U1.42 (GPIO4): now also J4.7 (Pin_7)
- net at U1.43 (GPIO5): now also J4.6 (Pin_6)
- net at U1.44 (GPIO6): now also J4.5 (Pin_5)
- net at U1.45 (GPIO7): now also J4.4 (Pin_4)
- net at U1.46 (GPIO8): now also J4.3 (Pin_3)
- net at U1.47 (GPIO9): now also J4.2 (Pin_2)
Changed lines of the file:
@@
 	10800 4850 10850 4850
 $Comp
-L power:GND #PWR014
+L power:GND #PWR015
 U 1 1 5E4286FE
 P 12000 5150
-F 0 "#PWR014" H 12000 4900 50  0001 C CNN
+F 0 "#PWR015" H 12000 4900 50  0001 C CNN
 F 1 "GND" H 12005 4977 50  0000 C CNN
 F 2 "" H 12000 5150 50  0001 C CNN
@@
 $EndComp
 $Comp
-L power:VPP #PWR03
+L power:VPP #PWR01
 U 1 1 5E42E243
 P 3700 1200
-F 0 "#PWR03" H 3700 1050 50  0001 C CNN
+F 0 "#PWR01" H 3700 1050 50  0001 C CNN
 F 1 "VPP" H 3715 1373 50  0000 C CNN
 F 2 "" H 3700 1200 50  0001 C CNN
@@
 $EndComp
 $Comp
-L power:GND #PWR016
+L power:GND #PWR017
 U 1 1 5E434956
 P 12150 4100
-F 0 "#PWR016" H 12150 3850 50  0001 C CNN
+F 0 "#PWR017" H 12150 3850 50  0001 C CNN
 F 1 "GND" H 12155 3927 50  0000 C CNN
 F 2 "" H 12150 4100 50  0001 C CNN
@@
 $EndComp
 $Comp
-L power:VPP #PWR020
+L power:VPP #PWR021
 U 1 1 5E43560E
 P 12550 3600
-F 0 "#PWR020" H 12550 3450 50  0001 C CNN
+F 0 "#PWR021" H 12550 3450 50  0001 C CNN
 F 1 "VPP" H 12565 3773 50  0000 C CNN
 F 2 "" H 12550 3600 50  0001 C CNN
@@
 $EndComp
 $Comp
-L power:VCC #PWR013
+L power:VCC #PWR014
 U 1 1 5E44BAC3
 P 12000 4500
-F 0 "#PWR013" H 12000 4350 50  0001 C CNN
+F 0 "#PWR014" H 12000 4350 50  0001 C CNN
 F 1 "VCC" H 12017 4673 50  0000 C CNN
 F 2 "" H 12000 4500 50  0001 C CNN
@@
 Connection ~ 12000 4550
 $Comp
-L Connector:Conn_01x01_Male J6
+L Connector:Conn_01x01_Male J7
 U 1 1 5E45417D
 P 12650 5550
-F 0 "J6" H 12622 5482 50  0000 R CNN
+F 0 "J7" H 12622 5482 50  0000 R CNN
 F 1 "Conn_01x01_Male" H 12622 5573 50  0000 R CNN
 F 2 "Connector_PinHeader_2.54mm:PinHeader_1x01_P2.54mm_Vertical" H 12650 5550 50  0001 C CNN
@@
 	11300 5300 11300 5550
 $Comp
-L power:VCC #PWR021
+L power:VCC #PWR022
 U 1 1 5E4581B1
 P 12600 5300
-F 0 "#PWR021" H 12600 5150 50  0001 C CNN
+F 0 "#PWR022" H 12600 5150 50  0001 C CNN
 F 1 "VCC" H 12617 5473 50  0000 C CNN
 F 2 "" H 12600 5300 50  0001 C CNN
@@
 	12200 5550 12450 5550
 $Comp
-L power:GND #PWR019
+L power:GND #PWR020
 U 1 1 5E3F2FC1
 P 12300 6650
-F 0 "#PWR019" H 12300 6400 50  0001 C CNN
+F 0 "#PWR020" H 12300 6400 50  0001 C CNN
 F 1 "GND" H 12305 6477 50  0000 C CNN
 F 2 "" H 12300 6650 50  0001 C CNN
@@
 	11550 5700 11550 5750
 $Comp
-L Connector:Conn_01x05_Male J5
+L Connector:Conn_01x05_Male J6
 U 1 1 5E3EE413
 P 12550 6400
-F 0 "J5" H 12522 6332 50  0000 R CNN
+F 0 "J6" H 12522 6332 50  0000 R CNN
 F 1 "Conn_01x05_Male" H 12522 6423 50  0000 R CNN
 F 2 "Connector_PinHeader_2.54mm:PinHeader_1x05_P2.54mm_Vertical" H 12550 6400 50  0001 C CNN
@@
 	11250 6100 12100 6100
 $Comp
-L Connector:Conn_01x03_Male J4
+L Connector:Conn_01x03_Male J5
 U 1 1 5E41D36A
 P 12550 5900
-F 0 "J4" H 12522 5832 50  0000 R CNN
+F 0 "J5" H 12522 5832 50  0000 R CNN
 F 1 "Conn_01x03_Male" H 12522 5923 50  0000 R CNN
 F 2 "Connector_PinHeader_2.54mm:PinHeader_1x03_P2.54mm_Vertical" H 12550 5900 50  0001 C CNN
@@
 	12100 5900 12100 6100
 $Comp
-L power:GND #PWR018
+L power:GND #PWR019
 U 1 1 5E41FB04
 P 12300 6050
-F 0 "#PWR018" H 12300 5800 50  0001 C CNN
+F 0 "#PWR019" H 12300 5800 50  0001 C CNN
 F 1 "GND" H 12305 5877 50  0000 C CNN
 F 2 "" H 12300 6050 50  0001 C CNN
@@
 $EndComp
 $Comp
-L power:VCC #PWR017
+L power:VCC #PWR018
 U 1 1 5E4203CF
 P 12300 5750
-F 0 "#PWR017" H 12300 5600 50  0001 C CNN
+F 0 "#PWR018" H 12300 5600 50  0001 C CNN
 F 1 "VCC" H 12317 5923 50  0000 C CNN
 F 2 "" H 12300 5750 50  0001 C CNN
@@
 $EndComp
 $Comp
-L power:GND #PWR02
+L power:GND #PWR03
 U 1 1 5E411FFA
 P 7600 10400
-F 0 "#PWR02" H 7600 10150 50  0001 C CNN
+F 0 "#PWR03" H 7600 10150 50  0001 C CNN
 F 1 "GND" H 7605 10227 50  0000 C CNN
 F 2 "" H 7600 10400 50  0001 C CNN
@@
 $EndComp
 $Comp
-L power:GND #PWR01
+L power:GND #PWR02
 U 1 1 5E473FEE
 P 5600 10100
-F 0 "#PWR01" H 5600 9850 50  0001 C CNN
+F 0 "#PWR02" H 5600 9850 50  0001 C CNN
 F 1 "GND" H 5605 9927 50  0000 C CNN
 F 2 "" H 5600 10100 50  0001 C CNN
@@
 $EndComp
 $Comp
-L power:GND #PWR022
+L power:GND #PWR023
 U 1 1 5EA009D1
 P 12750 2300
-F 0 "#PWR022" H 12750 2050 50  0001 C CNN
+F 0 "#PWR023" H 12750 2050 50  0001 C CNN
 F 1 "GND" H 12755 2127 50  0000 C CNN
 F 2 "" H 12750 2300 50  0001 C CNN
@@
 $EndComp
 $Comp
-L power:GND #PWR015
+L power:GND #PWR016
 U 1 1 5EA012A6
 P 12050 2300
-F 0 "#PWR015" H 12050 2050 50  0001 C CNN
+F 0 "#PWR016" H 12050 2050 50  0001 C CNN
 F 1 "GND" H 12055 2127 50  0000 C CNN
 F 2 "" H 12050 2300 50  0001 C CNN
@@
 $EndComp
 $Comp
-L power:GND #PWR024
+L power:GND #PWR025
 U 1 1 5EE76FDB
 P 14650 1350
-F 0 "#PWR024" H 14650 1100 50  0001 C CNN
+F 0 "#PWR025" H 14650 1100 50  0001 C CNN
 F 1 "GND" H 14655 1177 50  0000 C CNN
 F 2 "" H 14650 1350 50  0001 C CNN
@@
 	14650 1250 14650 1350
 $Comp
-L Connector:Conn_01x03_Male J7
+L Connector:Conn_01x03_Male J9
 U 1 1 5EFAA969
 P 13700 1950
-F 0 "J7" H 13672 1882 50  0000 R CNN
+F 0 "J9" H 13672 1882 50  0000 R CNN
 F 1 "Conn_01x03_Male" H 13672 1973 50  0000 R CNN
 F 2 "Connector_PinHeader_2.54mm:PinHeader_1x03_P2.54mm_Vertical" H 13700 1950 50  0001 C CNN
@@
 	13050 1950 13500 1950
 $Comp
-L power:GND #PWR023
+L power:GND #PWR024
 U 1 1 5F045204
 P 13450 2150
-F 0 "#PWR023" H 13450 1900 50  0001 C CNN
+F 0 "#PWR024" H 13450 1900 50  0001 C CNN
 F 1 "GND" H 13455 1977 50  0000 C CNN
 F 2 "" H 13450 2150 50  0001 C CNN
@@
 $EndComp
 $Comp
-L Connector:Conn_01x01_Male J9
+L Connector:Conn_01x01_Male J10
 U 1 1 5E678B51
 P 15700 800
-F 0 "J9" H 15672 732 50  0000 R CNN
+F 0 "J10" H 15672 732 50  0000 R CNN
 F 1 "Conn_01x01_Male" H 15672 823 50  0000 R CNN
 F 2 "TestPoint:TestPoint_Pad_4.0x4.0mm" H 15700 800 50  0001 C CNN
@@
 	9250 1200 9250 1300
 $Comp
-L power:VCC #PWR025
+L power:VCC #PWR026
 U 1 1 5EDCE56E
 P 15350 1150
-F 0 "#PWR025" H 15350 1000 50  0001 C CNN
+F 0 "#PWR026" H 15350 1000 50  0001 C CNN
 F 1 "VCC" H 15367 1323 50  0000 C CNN
 F 2 "" H 15350 1150 50  0001 C CNN
@@
 Wire Wire Line
 	3700 1350 3500 1350
+$Comp
+L Connector:Conn_01x08_Male J4
+U 1 1 5E73A265
+P 11950 7800
+F 0 "J4" H 11922 7682 50  0000 R CNN
+F 1 "Conn_01x08_Male" H 11922 7773 50  0000 R CNN
+F 2 "Connector_PinHeader_2.54mm:PinHeader_1x08_P2.54mm_Vertical" H 11950 7800 50  0001 C CNN
+F 3 "~" H 11950 7800 50  0001 C CNN
+	1    11950 7800
+	-1   0    0    1
+$EndComp
+Wire Wire Line
+	10800 7400 11750 7400
+Wire Wire Line
+	10800 7500 11750 7500
+Wire Wire Line
+	10800 7600 11750 7600
+Wire Wire Line
+	10800 7700 11750 7700
+Wire Wire Line
+	10800 7800 11750 7800
+Wire Wire Line
+	10800 7900 11750 7900
+Wire Wire Line
+	10800 8000 11750 8000
+$Comp
+L power:GND #PWR013
+U 1 1 5E95FE81
+P 11700 8150
+F 0 "#PWR013" H 11700 7900 50  0001 C CNN
+F 1 "GND" H 11705 7977 50  0000 C CNN
+F 2 "" H 11700 8150 50  0001 C CNN
+F 3 "" H 11700 8150 50  0001 C CNN
+	1    11700 8150
+	1    0    0    -1
+$EndComp
+Wire Wire Line
+	11750 8100 11700 8100
+Wire Wire Line
+	11700 8100 11700 8150
 $EndSCHEMATC

Commit message: First Version (Ordered)
Parts:
- removed J9: Conn_01x03_Male, Connector_PinHeader_2.54mm:PinHeader_1x03_P2.54mm_Vertical, symbol Connector:Conn_01x03_Male
- added J9: Conn_01x04_Male, Connector_PinHeader_2.54mm:PinHeader_1x04_P2.54mm_Vertical, symbol Connector:Conn_01x04_Male
- added Q19: IPT012N08N5, Package_TO_SOT_SMD:Infineon_PG-HSOF-8-1, symbol Transistor_FET:IPT012N08N5
- added R60: 4k7, Resistor_SMD:R_0805_2012Metric_Pad1.15x1.40mm_HandSolder, symbol Device:R
- added R61: 200, Resistor_SMD:R_0805_2012Metric_Pad1.15x1.40mm_HandSolder, symbol Device:R
- renumbered Q19 to Q20, Q20 to Q21, Q21 to Q22, R60 to R62, R61 to R63, R62 to R64, R63 to R65, R64 to R66, R65 to R67
Connections:
- net GND: now also J2.10 (Pin_10), R18.2, R38.2, J9.1 (Pin_1), R60.2; no longer R38.1, U1.38 (C0)
- net at Q21.3 (D): now also Q19.3 (D); no longer U2.4 (IP+)
- net at R67.1: now also J9.4 (Pin_4)
- net at R63.1: now also J9.3 (Pin_3)
- new net: R38.1, U1.38 (C0)
- new net: Q19.2 (S), U2.4 (IP+)
- new net: Q19.1 (G), R60.1, R61.2
- new net: J9.2 (Pin_2), R61.1
Other:
- moved on the sheet: J3, U2
